File: BMS_Teidesat/BMS_Teidesat.kicad_sch (KiCad schematic)
At the start: 50 parts, among them J1 Battery, J2 Battery, U1 AD8605ACBZ-REEL7, U2 AD8606ARMZ-REEL, U3 ADA4940-1ACPZ-R7, U4 ACS37002LMCATR-050B5, U5 AD7091R-8BCPZ-RL7, U6 CSD86311W1723, U7 AD8605ACBZ-REEL7, U8 STM32G474VET6, U9 TMS5703137DPGEQQ1

Commit message: Nuevo circuito de potencia
Hemos tenido que rediseñar el circuito de potencia, añadiendo nuevos MOSFETS y drivers para dividir la corriente entre 3 y evitar problemas de sobrecalentamiento

Co-Authored-By: hugohdezmo <238262256+hugohdezmo@users.noreply.github.com>
Parts:
- removed J2: Battery, Connector_PinSocket_1.00mm:PinSocket_1x02_P1.00mm_Vertical_SMD_Pin1Left, symbol Connector:Conn_01x02_Pin
- removed R20: 10, Resistor_SMD:R_0201_0603Metric, symbol Device:R
- removed U6: CSD86311W1723, Huellas BMS:BGA12C50P4X3_228X170X62, symbol CSD86311W1723:CSD86311W1723
- removed U8: STM32G474VET6, Huellas BMS:QFP50P1600X1600X160-100N, symbol STM32G474VET6:STM32G474VET6
- added C5, C6, C7, C8: 10n, Capacitor_SMD:C_0805_2012Metric, symbol Device:C
- added D3, D4, D5, D6: SS14, Huellas BMS:DIOM6859X262N, symbol Diode:SS14
- added R10, R22, R23, R25, R26, R27, R28, R29, R30, R8, R9: 10, Resistor_SMD:R_0201_0603Metric, symbol Device:R
- added U1, U13: MCP1407-E_SN, Huellas BMS:SOIC127P600X175-8N, symbol MCP1407-E_SN:MCP1407-E_SN
- added U10, U11, U12, U4, U5, U6: IPT004N03L, Huellas BMS:PG-HSOF-8-1, symbol IPT004N03L:IPT004N03L
- D1, D2: footprint Huellas BMS:DIOM8059X256N -> Huellas BMS:DIOM6859X262N
- renumbered C5 to C10, C6 to C11, C7 to C12, C8 to C13, R10 to R11, R11 to R12, R9 to R13, R12 to R14, R13 to R15, R14 to R16, R15 to R17, R16 to R18, R17 to R19, R18 to R20, R19 to R24, R5 to R31, R6 to R5, R7 to R6, R8 to R7, U5 to U14, U7 to U15, U1 to U3, U3 to U7, U4 to U8
Connections:
- net +3V3: no longer H2.27 (Pin_27), H2.28 (Pin_28)
- net +5V: now also U1.1 (VDD_1), U1.8 (VDD_2), U13.1 (VDD_1), U13.8 (VDD_2); no longer H2.25 (Pin_25), H2.26 (Pin_26)
- net CLOCK MC: now also U9.95 (MIBSPI1CLK)
- net CONTROL1: now also U9.16 (GIOA[6]), U1.2 (INPUT)
- net CONTROL2: now also U9.22 (GIOA[7]), U13.2 (INPUT)
- net CS: now also U9.105 (MIBSPI1NCS[0])
- net GIOA: now also U9.9 (GIOA[2])
- net GND: now also U1.4 (GND_1), U1.5 (GND_2), U13.4 (GND_1), U13.5 (GND_2); no longer H2.21 (Pin_21), H2.22 (Pin_22), H2.29 (Pin_29), H2.30 (Pin_30), H2.31 (Pin_31), H2.32 (Pin_32)
- net MOSI MC: now also U9.93 (MIBSPI1SIMO)
- net OUT CAD: now also U9.94 (MIBSPI1SOMI)
- net RESET: now also U9.14 (GIOA[5])
- net BATTERY: now reaches C3.1
- net BATTERY: now also C4.1, D1.1 (K), D2.1 (K), J1.1 (Pin_1), R1.1, C5.1, D3.1 (K), U4.9 (D), U5.9 (D), U6.9 (D); no longer D1.2 (A)
- net at C3.2: now also R21.1
- net at C4.2: now also R22.1; no longer R21.1
- net +BATT: no longer names the net of H2.45 (Pin_45)
- net +BATT: no longer H2.46 (Pin_46)
- net +BATTERY renamed CURRENT S
- net CURRENT S: now also D3.2 (A), R22.2, U6.2 (S_1), U6.3 (S_2), U6.4 (S_3), U6.5 (S_4), U6.6 (S_5), U6.7 (S_6), U6.8 (S_7); no longer D1.1 (K), D2.1 (K), R21.2
- net +LOAD renamed MOSFET3
- net MOSFET3: now also D6.2 (A), R27.2, U12.2 (S_1), U12.3 (S_2), U12.4 (S_3), U12.5 (S_4), U12.6 (S_5), U12.7 (S_6), U12.8 (S_7)
- net EPS renamed MOSFET2
- net MOSFET2: now also R21.2, D5.2 (A), R26.2, U11.2 (S_1), U11.3 (S_2), U11.4 (S_3), U11.5 (S_4), U11.6 (S_5), U11.7 (S_6), U11.8 (S_7), U5.2 (S_1), U5.3 (S_2), U5.4 (S_3), U5.5 (S_4), U5.6 (S_5), U5.7 (S_6), U5.8 (S_7); no longer C4.1
- new net: C5.2, R23.1
- new net: C8.1, D6.1 (K), U12.9 (D)
- new net: R10.1, R8.1, R9.1, U1.6 (OUT_1), U1.7 (OUT_2)
- new net: R8.2, U4.1 (G)
- new net: C8.2, R27.1
- new net: R28.1, R29.1, R30.1, U13.6 (OUT_1), U13.7 (OUT_2)
- new net: R28.2, U10.1 (G)
- new net: C6.1, D4.1 (K), U10.9 (D)
- new net: R30.2, U12.1 (G)
- new net: C6.2, R25.1
- new net: R9.2, U5.1 (G)
- new net: C7.2, R26.1
- new net: R10.2, U6.1 (G)
- new net: R29.2, U11.1 (G)
- new net: C7.1, D5.1 (K), U11.9 (D)
- new net MOSFET1: D1.2 (A), D4.2 (A), R23.2, R25.2, U10.2 (S_1), U10.3 (S_2), U10.4 (S_3), U10.5 (S_4), U10.6 (S_5), U10.7 (S_6), U10.8 (S_7), U4.2 (S_1), U4.3 (S_2), U4.4 (S_3), U4.5 (S_4), U4.6 (S_5), U4.7 (S_6), U4.8 (S_7)
- no-connect marks 356 -> 254
Other:
- note added: "Driver"
- note added: "Red Snubber"
- note removed: "C Snubber"
- note removed: "Diodo C.R"
- note removed: "Es importante que fisicamente esten cerca del transistor"
- note removed: "Los valores actuales son una recomendación"
- note removed: "MICROCONTROLADOR (Teidesat)"
- note removed: "Para el calculo de las R y C en la red de Snubber es necesario medir los picos de voltaje de la placa mientras se apagan los mosfet con un osciloscopio y calcular los valores de R y C usando esa medida"
- note removed: "R Snubber"
- moved on the sheet: C1, C9, J1, R1, R13, R14, R16, R17, R18, R19, R20, R24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
